File: TramController.sch (KiCad schematic (older format))
At the start: 31 parts, among them J1 Screw_Terminal_01x04, J2 power, J3 Screw_Terminal_01x04, J4 servo, J5 servo, J6 power, K1 SANYOU_SRD_Form_C, Q1 BC547, U1 EL814, U2 L298HN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

Commit message: replaced schematic with a more up to date one
Parts:
- added C10, C6, C7, C8: 100nF, Capacitor_THT:C_Disc_D3.0mm_W1.6mm_P2.50mm, symbol Device:C
- added C9: 1000uF, Capacitor_THT:CP_Radial_D8.0mm_P3.50mm, symbol Device:CP
- added JP1, JP2, JP3: jmp, symbol Jumper:SolderJumper_2_Open
- added R5: 4k7, Resistor_THT:R_Axial_DIN0204_L3.6mm_D1.6mm_P7.62mm_Horizontal, symbol Device:R
- C1: value CP -> 1000uF
- C2: value C -> 100nF
- J1: value Screw_Terminal_01x04 -> to Tracks
- J3: value Screw_Terminal_01x04 -> control panel
- K1: value SANYOU_SRD_Form_C -> SPST
- R1: value R -> 1k
- R2, R3: value R -> 1R
- R7: value R -> 33R
Connections:
- net labels added: JP1, JP2, JP3, frontTrack, rearTrack, redIn, redOut, relayPin, shortCircuit, slidings
- net labels removed: currentSense, front, rear, red
- wire segments 140 -> 151
- no-connect marks 17 -> 10
Other:
- note added: "servo's for points\n"
- note added: "shunt resistors\n"
- note added: "switch between 1 of 2 tracks\n"
- note added: "to H-bridge"
- note added: "to side tracks for\ncurrent sense"
- note added: "voltage drop for undetected track"
- moved on the sheet: A1, C1, C2, C3, C4, C5, D1, D2, D3, D4, J1, J2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
